File: kicad/MIDI_controller/MIDI_controller.kicad_sch (KiCad schematic)
At the start: 26 parts, among them J1 AVR-ISP-6, J2 DIN-5, J3 Jack-DC, SW1 RotaryEncoder_Switch, SW10 RotaryEncoder_Switch, SW11 RotaryEncoder_Switch, SW12 RotaryEncoder_Switch, SW2 RotaryEncoder_Switch, SW3 RotaryEncoder_Switch, SW4 RotaryEncoder_Switch, SW5 RotaryEncoder_Switch, SW6 RotaryEncoder_Switch, SW7 RotaryEncoder_Switch, SW8 RotaryEncoder_Switch, SW9 RotaryEncoder_Switch, U1 ATmega328P-P, U2 MCP23017_SP, U3 MCP23017_SP, U4 MCP23017_SP, U5 LM317_TO-220, Y1 Crystal

Commit message: small update schematic
Parts:
- removed SW10, SW11, SW12, SW2, SW3, SW4, SW5, SW6, SW7, SW8, SW9: RotaryEncoder_Switch, symbol Device:RotaryEncoder_Switch
Connections:
- net GND: now also C1.2, C2.2, SW1.C, SW1.S2; no longer C1.1, C2.1
- net VCC: now also SW1.A, SW1.S1
- net at C4.1, U5.2 (VO): no longer U1.7 (VCC)
- net EXP1/GPB1: now reaches SW1.B
- new net: C2.1, U1.9 (XTAL1/PB6), Y1.2
- new net: C1.1, U1.10 (XTAL2/PB7), Y1.1
Other:
- moved on the sheet: C1, C2, J3, Y1

Commit message: update kicad schematic
Parts:
- removed U5: LM317_TO-220, Package_TO_SOT_THT:TO-220-3_Vertical, symbol Regulator_Linear:LM317_TO-220
- added R1: 10kΩ, symbol Device:R
- added SW10, SW11, SW12, SW2, SW3, SW4, SW5, SW6, SW7, SW8, SW9: RotaryEncoder_Switch, symbol Device:RotaryEncoder_Switch
- added U5: AMS1117-5.0, Package_TO_SOT_SMD:SOT-223-3_TabPin2, symbol Regulator_Linear:AMS1117-5.0
- C1, C2, C4: value C -> 22μF
- C3: value C -> 10μF
- Y1: value Crystal -> Crystal 16MHz
Connections:
- net EXP1/GPB1 is gone; now on net +5V: SW1.B
- net GND: now also Brd1.1 (GND), J1.6 (GND), U1.22 (GND), U1.8 (GND), U2.10 (VSS), U2.15 (A0), U2.16 (A1), U2.17 (A2), U3.10 (VSS), U3.16 (A1), U3.17 (A2), U4.10 (VSS), U4.15 (A0), U4.17 (A2), SW10.C, SW10.S2, SW11.C, SW11.S2, SW12.C, SW12.S2, SW2.C, SW2.S2, SW3.C, SW3.S2, SW4.C, SW4.S2, SW5.C, SW5.S2, SW6.C, SW6.S2, SW7.C, SW7.S2, SW8.C, SW8.S2, SW9.C, SW9.S2; no longer C3.2, C4.2
- net +5V: now reaches C4.1
- net +5V: now also Brd1.2 (VCC), J1.2 (VCC), SW1.A, SW1.S1, U1.20 (AVCC), U1.7 (VCC), U2.1 (GPB0), U2.2 (GPB1), U2.21 (GPA0), U2.22 (GPA1), U2.23 (GPA2), U2.25 (GPA4), U2.26 (GPA5), U2.27 (GPA6), U2.3 (GPB2), U2.5 (GPB4), U2.6 (GPB5), U2.7 (GPB6), U2.9 (VDD), U3.1 (GPB0), U3.15 (A0), U3.2 (GPB1), U3.21 (GPA0), U3.22 (GPA1), U3.23 (GPA2), U3.25 (GPA4), U3.26 (GPA5), U3.27 (GPA6), U3.3 (GPB2), U3.5 (GPB4), U3.6 (GPB5), U3.7 (GPB6), U3.9 (VDD), U4.1 (GPB0), U4.16 (A1), U4.2 (GPB1), U4.21 (GPA0), U4.22 (GPA1), U4.23 (GPA2), U4.25 (GPA4), U4.26 (GPA5), U4.27 (GPA6), U4.3 (GPB2), U4.5 (GPB4), U4.6 (GPB5), U4.7 (GPB6), U4.9 (VDD), R1.2, SW10.A, SW10.B, SW10.S1, SW11.A, SW11.B, SW11.S1, SW12.A, SW12.B, SW12.S1, SW2.A, SW2.B, SW2.S1, SW3.A, SW3.B, SW3.S1, SW4.A, SW4.B, SW4.S1, SW5.A, SW5.B, SW5.S1, SW6.A, SW6.B, SW6.S1, SW7.A, SW7.B, SW7.S1, SW8.A, SW8.B, SW8.S1, SW9.A, SW9.B, SW9.S1, U5.2 (VO)
- net RST: now reaches U1.1 (~{RESET}/PC6)
- net RST: now also J1.5 (~{RST}), U2.18 (~{RESET}), U3.18 (~{RESET}), U4.18 (~{RESET}), R1.1
- net MOSI: now reaches U1.17 (PB3)
- net MOSI: now also J1.4 (MOSI)
- net MISO: now reaches U1.18 (PB4)
- net MISO: now also J1.1 (MISO)
- net SCK: now reaches U1.19 (PB5)
- net SCK: now also J1.3 (SCK)
- net SDA: now reaches U1.27 (PC4)
- net SDA: now also Brd1.4 (SDA), U2.13 (SDA), U3.13 (SDA), U4.13 (SDA)
- net SCL: now reaches U1.28 (PC5)
- net SCL: now also Brd1.3 (SCL), U2.12 (SCK), U3.12 (SCK), U4.12 (SCK)
- net at J3.1: now also C3.1, U5.3 (VI)
- net at J3.2: now also C3.2, C4.2, U5.1 (GND)
- removed net VCC: C3.1, SW1.A, SW1.S1
- no-connect marks 0 -> 19
Other:
- note added: "Encoders"
- note added: "Expanders"
- note added: "ISP"
- note added: "Microchip"
- note added: "OLED"
- note added: "Power supply"
- title: (none) -> MIDI Controller
- moved on the sheet: Brd1, C1, C2, C3, C4, J1, J2, J3, SW1, U1, U2, Y1

Commit message: schema midi
Parts:
- removed J2: DIN-5, symbol Connector:DIN-5
- removed SW1, SW10, SW11, SW12, SW2, SW3, SW4, SW5, SW6, SW7, SW8, SW9: RotaryEncoder_Switch, symbol Device:RotaryEncoder_Switch
- added D1: LED (RED), LED_THT:LED_D1.8mm_W3.3mm_H2.4mm, symbol Device:LED
- added J2: DIN-5_180degree, symbol Connector:DIN-5_180degree
- added R2: 220Ω, symbol Device:R
- added R3: 160Ω, symbol Device:R
- added SW1, SW10, SW11, SW12, SW2, SW3, SW4, SW5, SW6, SW7, SW8, SW9: RotaryEncoder_Switch_MP, Rotary_Encoder:RotaryEncoder_Alps_EC11E-Switch_Vertical_H20mm_MountingHoles, symbol Device:RotaryEncoder_Switch_MP
- Brd1: footprint (none) -> Connector_PinHeader_1.27mm:PinHeader_1x04_P1.27mm_Vertical
- J1: footprint (none) -> Connector_IDC:IDC-Header_2x03_P2.54mm_Vertical
- J3: footprint (none) -> Connector_PinHeader_1.27mm:PinHeader_1x02_P1.27mm_Vertical
- Y1: footprint (none) -> Crystal:Crystal_HC52-8mm_Vertical
Connections:
- net +5V: now also R2.1, SW1.A, SW1.B, SW1.S1, SW10.A, SW10.B, SW10.S1, SW11.A, SW11.B, SW11.S1, SW12.A, SW12.B, SW12.S1, SW2.A, SW2.B, SW2.S1, SW3.A, SW3.B, SW3.S1, SW4.A, SW4.B, SW4.S1, SW5.A, SW5.B, SW5.S1, SW6.A, SW6.B, SW6.S1, SW7.A, SW7.B, SW7.S1, SW8.A, SW8.B, SW8.S1, SW9.A, SW9.B, SW9.S1
- net GND: now also C3.2, C4.2, J3.2, U5.1 (GND), D1.1 (K), J2.2, SW1.C, SW1.S2, SW10.C, SW10.S2, SW11.C, SW11.S2, SW12.C, SW12.S2, SW2.C, SW2.S2, SW3.C, SW3.S2, SW4.C, SW4.S2, SW5.C, SW5.S2, SW6.C, SW6.S2, SW7.C, SW7.S2, SW8.C, SW8.S2, SW9.C, SW9.S2
- net TX: now reaches U1.3 (PD1)
- net TX: now also J2.5
- net at U1.6 (PD4): now also R3.1
- new net: J2.4, R2.2
- new net: D1.2 (A), R3.2
- no-connect marks 19 -> 46
Other:
- note added: "MIDI OUT"
- moved on the sheet: Brd1, C3, C4, J1, J3, U5

Commit message: small update schem
Parts:
- C1, C2: value 22μF -> 22pF ceramic
- C4: footprint (none) -> Capacitor_THT:CP_Radial_D4.0mm_P1.50mm
- SW1, SW10, SW11, SW12, SW2, SW3, SW4, SW5, SW6, SW7, SW8, SW9: footprint Rotary_Encoder:RotaryEncoder_Alps_EC11E-Switch_Vertical_H20mm_MountingHoles -> Rotary_Encoder:RotaryEncoder_Alps_EC11E-Switch_Vertical_H20mm
- U1, U2, U3, U4: footprint Package_DIP:DIP-28_W7.62mm -> Package_DIP:DIP-28_W7.62mm_LongPads
- Y1: footprint Crystal:Crystal_HC52-8mm_Vertical -> Crystal:Crystal_HC49-U_Vertical
Changed lines of the file:
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@@
 			)
 		)
-		(property "Footprint" "Rotary_Encoder:RotaryEncoder_Alps_EC11E-Switch_Vertical_H20mm_MountingHoles"
+		(property "Footprint" "Rotary_Encoder:RotaryEncoder_Alps_EC11E-Switch_Vertical_H20mm"
 			(at 259.08 23.876 0)
 			(effects
@@
 			)
 		)
-		(property "Value" "22μF"
-			(at 73.66 77.47 90)
+		(property "Value" "22pF ceramic"
+			(at 78.486 77.47 90)
 			(effects
 				(font
@@
 			)
 		)
-		(property "Footprint" "Rotary_Encoder:RotaryEncoder_Alps_EC11E-Switch_Vertical_H20mm_MountingHoles"
+		(property "Footprint" "Rotary_Encoder:RotaryEncoder_Alps_EC11E-Switch_Vertical_H20mm"
 			(at 170.18 23.876 0)
 			(effects
@@
 			)
 		)
-		(property "Footprint" ""
+		(property "Footprint" "Capacitor_THT:CP_Radial_D4.0mm_P1.50mm"
 			(at 67.0052 38.1 0)
 			(effects
@@
 			)
 		)
-		(property "Footprint" "Rotary_Encoder:RotaryEncoder_Alps_EC11E-Switch_Vertical_H20mm_MountingHoles"
+		(property "Footprint" "Rotary_Encoder:RotaryEncoder_Alps_EC11E-Switch_Vertical_H20mm"
 			(at 214.63 46.736 0)
 			(effects
@@
 			)
 		)
-		(property "Footprint" "Crystal:Crystal_HC52-8mm_Vertical"
+		(property "Footprint" "Crystal:Crystal_HC49-U_Vertical"
 			(at 64.77 86.36 0)
 			(effects
@@
 			)
 		)
-		(property "Footprint" "Rotary_Encoder:RotaryEncoder_Alps_EC11E-Switch_Vertical_H20mm_MountingHoles"
+		(property "Footprint" "Rotary_Encoder:RotaryEncoder_Alps_EC11E-Switch_Vertical_H20mm"
 			(at 214.63 23.876 0)
 			(effects
@@
 			)
 		)
-		(property "Footprint" "Rotary_Encoder:RotaryEncoder_Alps_EC11E-Switch_Vertical_H20mm_MountingHoles"
+		(property "Footprint" "Rotary_Encoder:RotaryEncoder_Alps_EC11E-Switch_Vertical_H20mm"
 			(at 259.08 70.866 0)
 			(effects
@@
 			)
 		)
-		(property "Footprint" "Package_DIP:DIP-28_W7.62mm"
+		(property "Footprint" "Package_DIP:DIP-28_W7.62mm_LongPads"
 			(at 31.75 100.33 0)
 			(effects
@@
 			)
 		)
-		(property "Footprint" "Rotary_Encoder:RotaryEncoder_Alps_EC11E-Switch_Vertical_H20mm_MountingHoles"
+		(property "Footprint" "Rotary_Encoder:RotaryEncoder_Alps_EC11E-Switch_Vertical_H20mm"
 			(at 170.18 46.736 0)
 			(effects
@@
 			)
 		)
-		(property "Footprint" "Rotary_Encoder:RotaryEncoder_Alps_EC11E-Switch_Vertical_H20mm_MountingHoles"
+		(property "Footprint" "Rotary_Encoder:RotaryEncoder_Alps_EC11E-Switch_Vertical_H20mm"
 			(at 259.08 46.736 0)
 			(effects
@@
 			)
 		)
-		(property "Footprint" "Package_DIP:DIP-28_W7.62mm"
+		(property "Footprint" "Package_DIP:DIP-28_W7.62mm_LongPads"
 			(at 156.21 114.3 0)
 			(effects
@@
 			)
 		)
-		(property "Value" "22μF"
+		(property "Value" "22pF ceramic"
 			(at 73.66 95.504 90)
 			(effects
@@
 					(size 1.27 1.27)
 				)
-				(justify left)
 			)
 		)
@@
 			)
 		)
-		(property "Footprint" "Rotary_Encoder:RotaryEncoder_Alps_EC11E-Switch_Vertical_H20mm_MountingHoles"
+		(property "Footprint" "Rotary_Encoder:RotaryEncoder_Alps_EC11E-Switch_Vertical_H20mm"
 			(at 125.73 46.736 0)
 			(effects
@@
 			)
 		)
-		(property "Footprint" "Rotary_Encoder:RotaryEncoder_Alps_EC11E-Switch_Vertical_H20mm_MountingHoles"
+		(property "Footprint" "Rotary_Encoder:RotaryEncoder_Alps_EC11E-Switch_Vertical_H20mm"
 			(at 170.18 70.866 0)
 			(effects
@@
 			)
 		)
-		(property "Footprint" "Package_DIP:DIP-28_W7.62mm"
+		(property "Footprint" "Package_DIP:DIP-28_W7.62mm_LongPads"
 			(at 273.05 114.3 0)
 			(effects
@@
 			)
 		)
-		(property "Footprint" "Package_DIP:DIP-28_W7.62mm"
+		(property "Footprint" "Package_DIP:DIP-28_W7.62mm_LongPads"
 			(at 214.63 114.3 0)
 			(effects
@@
 			)
 		)
-		(property "Footprint" "Rotary_Encoder:RotaryEncoder_Alps_EC11E-Switch_Vertical_H20mm_MountingHoles"
+		(property "Footprint" "Rotary_Encoder:RotaryEncoder_Alps_EC11E-Switch_Vertical_H20mm"
 			(at 125.73 23.876 0)
 			(effects
@@
 			)
 		)
-		(property "Footprint" "Rotary_Encoder:RotaryEncoder_Alps_EC11E-Switch_Vertical_H20mm_MountingHoles"
+		(property "Footprint" "Rotary_Encoder:RotaryEncoder_Alps_EC11E-Switch_Vertical_H20mm"
 			(at 214.63 70.866 0)
 			(effects
@@
 			)
 		)
-		(property "Footprint" "Rotary_Encoder:RotaryEncoder_Alps_EC11E-Switch_Vertical_H20mm_MountingHoles"
+		(property "Footprint" "Rotary_Encoder:RotaryEncoder_Alps_EC11E-Switch_Vertical_H20mm"
 			(at 125.73 70.866 0)
 			(effects

Commit message: update capacitor schem
Parts:
- removed D1: LED (RED), LED_THT:LED_D1.8mm_W3.3mm_H2.4mm, symbol Device:LED
- removed R3: 160Ω, symbol Device:R
- added C5, C6, C7, C8, C9: 0.1uF (100nF) ceramic, Capacitor_THT:C_Disc_D5.0mm_W2.5mm_P5.00mm, symbol Device:C
- added TP1, TP2, TP3: TestPoint, symbol Connector:TestPoint
Connections:
- net GND: now also TP3.1
- net SCL: now also TP2.1
- net SDA: now also TP1.1
- no-connect marks 46 -> 47

Commit message: update schem
Parts:
- removed C3: 10μF, symbol Device:C
- removed C4: 22μF, Capacitor_THT:CP_Radial_D4.0mm_P1.50mm, symbol Device:C
- removed C6: 0.1uF (100nF) ceramic, Capacitor_THT:C_Disc_D5.0mm_W2.5mm_P5.00mm, symbol Device:C
- added C3: 10uF, symbol Device:C_Polarized
- added C4: 22uF, symbol Device:C_Polarized
- C1, C2: value 22pF ceramic -> 22pF
- C5, C7, C8, C9: value 0.1uF (100nF) ceramic -> 0.1uF (100nF)
Connections:
- net +5V: now also C5.1, C7.1, C8.1, C9.1, C4.1; no longer J1.2 (VCC)
- net GND: now also C5.2, C7.2, C8.2, C9.2, C3.2, C4.2; no longer J1.6 (GND)
- net SCL: no longer TP2.1
- net at U1.6 (PD4): now also TP2.1
- net at J3.1, U5.3 (VI): now also C3.1
- no-connect marks 47 -> 48
Other:
- note added: "I2c address"
- moved on the sheet: Brd1, C1, C2, C5, C7, R1, SW1, SW10, SW11, SW12, SW2, SW3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

Commit message: routing test code and update schematics with interrupts
Connections:
- net at TP2.1: now also U1.4 (PD2); no longer U1.6 (PD4)
- net INT1: now reaches U1.11 (PD5)
- net INT1: now also U2.20 (INTA)
- net INT2: now reaches U1.12 (PD6)
- net INT2: now also U3.20 (INTA)
- net INT3: now reaches U1.13 (PD7)
- net INT3: now also U4.20 (INTA)
- no-connect marks 48 -> 42
Other:
- moved on the sheet: TP2
Changed lines of the file:
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@@
 	)
 	(no_connect
-		(at 46.99 119.38)
-	)
-	(no_connect
 		(at 205.74 139.7)
 	)
@@
 	)
 	(no_connect
-		(at 104.14 127)
-	)
-	(no_connect
 		(at 46.99 99.06)
 	)
@@
 	)
 	(no_connect
-		(at 233.68 127)
-	)
-	(no_connect
 		(at 233.68 124.46)
 	)
@@
 	)
 	(no_connect
-		(at 46.99 127)
-	)
-	(no_connect
 		(at 269.24 129.54)
 	)
@@
 	)
 	(no_connect
-		(at 170.18 127)
-	)
-	(no_connect
 		(at 172.72 81.28)
 	)
@@
 	)
 	(no_connect
+		(at 46.99 124.46)
+	)
+	(no_connect
 		(at 16.51 71.12)
 	)
@@
 	)
 	(no_connect
-		(at 46.99 129.54)
-	)
-	(no_connect
 		(at 139.7 116.84)
 	)
@@
 	)
 	(no_connect
-		(at 46.99 132.08)
-	)
-	(no_connect
 		(at 217.17 81.28)
 	)
@@
 	(wire
 		(pts
+			(xy 46.99 119.38) (xy 50.8 119.38)
+		)
+		(stroke
+			(width 0)
+			(type default)
+		)
+	)
+	(wire
+		(pts
 			(xy 142.24 142.24) (xy 139.7 142.24)
 		)
@@
 	(wire
 		(pts
-			(xy 46.99 124.46) (xy 50.8 124.46)
-		)
-		(stroke
-			(width 0)
-			(type default)
-		)
-	)
-	(wire
-		(pts
 			(xy 157.48 25.4) (xy 165.1 25.4)
 		)
@@
 	(wire
 		(pts
+			(xy 46.99 129.54) (xy 53.34 129.54)
+		)
+		(stroke
+			(width 0)
+			(type default)
+		)
+	)
+	(wire
+		(pts
 			(xy 55.88 34.29) (xy 55.88 40.64)
 		)
@@
 	(wire
 		(pts
+			(xy 167.64 127) (xy 170.18 127)
+		)
+		(stroke
+			(width 0)
+			(type default)
+		)
+	)
+	(wire
+		(pts
 			(xy 227.33 59.69) (xy 252.73 59.69)
 		)
@@
 	(wire
 		(pts
+			(xy 46.99 132.08) (xy 53.34 132.08)
+		)
+		(stroke
+			(width 0)
+			(type default)
+		)
+	)
+	(wire
+		(pts
 			(xy 31.75 63.5) (xy 31.75 62.23)
 		)
@@
 	(wire
 		(pts
+			(xy 46.99 127) (xy 53.34 127)
+		)
+		(stroke
+			(width 0)
+			(type default)
+		)
+	)
+	(wire
+		(pts
 			(xy 31.75 139.7) (xy 31.75 140.97)
 		)
@@
 	(wire
 		(pts
+			(xy 101.6 127) (xy 104.14 127)
+		)
+		(stroke
+			(width 0)
+			(type default)
+		)
+	)
+	(wire
+		(pts
 			(xy 110.49 48.26) (xy 113.03 48.26)
 		)
@@
 	(wire
 		(pts
+			(xy 231.14 127) (xy 233.68 127)
+		)
+		(stroke
+			(width 0)
+			(type default)
+		)
+	)
+	(wire
+		(pts
 			(xy 243.84 53.34) (xy 250.19 53.34)
 		)
@@
 		)
 	)
+	(label "INT1"
+		(at 53.34 127 0)
+		(effects
+			(font
+				(size 1.27 1.27)
+				(thickness 0.254)
+				(bold yes)
+			)
+			(justify left bottom)
+		)
+	)
+	(label "INT2"
+		(at 53.34 129.54 0)
+		(effects
+			(font
+				(size 1.27 1.27)
+				(thickness 0.254)
+				(bold yes)
+			)
+			(justify left bottom)
+		)
+	)
+	(label "INT3"
+		(at 231.14 127 180)
+		(effects
+			(font
+				(size 1.27 1.27)
+				(thickness 0.254)
+				(bold yes)
+			)
+			(justify right bottom)
+		)
+	)
 	(label "CLK12"
 		(at 271.78 142.24 0)
@@
 		)
 	)
+	(label "INT3"
+		(at 53.34 132.08 0)
+		(effects
+			(font
+				(size 1.27 1.27)
+				(thickness 0.254)
+				(bold yes)
+			)
+			(justify left bottom)
+		)
+	)
 	(label "SDA"
 		(at 231.14 109.22 180)
@@
 		)
 	)
+	(label "INT1"
+		(at 101.6 127 180)
+		(effects
+			(font
+				(size 1.27 1.27)
+				(thickness 0.254)
+				(bold yes)
+			)
+			(justify right bottom)
+		)
+	)
 	(label "SW1"
 		(at 142.24 114.3 0)
@@
 		)
 	)
+	(label "INT2"
+		(at 167.64 127 180)
+		(effects
+			(font
+				(size 1.27 1.27)
+				(thickness 0.254)
+				(bold yes)
+			)
+			(justify right bottom)
+		)
+	)
 	(label "SW5"
 		(at 140.97 48.26 0)
@@
 	(symbol
 		(lib_id "Connector:TestPoint")
-		(at 50.8 124.46 270)
+		(at 50.8 119.38 270)
 		(unit 1)
 		(exclude_from_sim no)
@@
 		(fields_autoplaced yes)
 		(property "Reference" "TP2"
-			(at 55.88 123.1899 90)
+			(at 55.88 118.1099 90)
 			(effects
 				(font
@@
 		)
 		(property "Value" "TestPoint"
-			(at 55.88 125.7299 90)
+			(at 55.88 120.6499 90)
 			(effects
 				(font
@@
 		)
 		(property "Footprint" ""
-			(at 50.8 129.54 0)
+			(at 50.8 124.46 0)
 			(effects
 				(font
@@
 		)
 		(property "Datasheet" "~"
-			(at 50.8 129.54 0)
+			(at 50.8 124.46 0)
 			(effects
 				(font
@@
 		)
 		(property "Description" "test point"
-			(at 50.8 124.46 0)
+			(at 50.8 119.38 0)
 			(effects
 				(font
